File: Dakboard-HDMI-dimmer-HW-KiCAD/Mainboard v1/Mainboard v1.kicad_sch (KiCad schematic)
At the start: 0 parts

Commit message: schematic, BOM, board wip
Parts:
- added C2, C5: 10 uF, Capacitor_SMD:C_0805_2012Metric_Pad1.18x1.45mm_HandSolder, symbol Device:C
- added C3, C4: 100 nF, Capacitor_SMD:C_0805_2012Metric_Pad1.18x1.45mm_HandSolder, symbol Device:C
- added J1: Conn_02x20_Odd_Even, Connector_PinSocket_2.54mm:PinSocket_2x20_P2.54mm_Vertical, symbol Connector_Generic:Conn_02x20_Odd_Even
- added J2: Conn_01x05, Connector_PinHeader_2.54mm:PinHeader_1x05_P2.54mm_Horizontal, symbol Connector_Generic:Conn_01x05
- added J3: Conn_01x03, Connector_PinHeader_2.54mm:PinHeader_1x03_P2.54mm_Horizontal, symbol Connector_Generic:Conn_01x03
- added R1: 100K, Resistor_SMD:R_0805_2012Metric_Pad1.20x1.40mm_HandSolder, symbol Device:R
- added R2, R3: 47R, Resistor_SMD:R_0805_2012Metric_Pad1.20x1.40mm_HandSolder, symbol Device:R
- added R4, R5: 4K7, Resistor_SMD:R_0805_2012Metric_Pad1.20x1.40mm_HandSolder, symbol Device:R
- added R6: 1K, Resistor_SMD:R_0805_2012Metric_Pad1.20x1.40mm_HandSolder, symbol Device:R
Connections:
- new net: J3.2 (Pin_2), R6.2
- new net: J2.3 (Pin_3), R2.2, R4.2
- new net: J2.4 (Pin_4), R3.2, R5.2
- new net +3V3: C2.2, C3.2, J1.1 (Pin_1), J1.17 (Pin_17), J2.1 (Pin_1), R4.1, R5.1
- new net +5V: C4.2, C5.2, J1.2 (Pin_2), J1.4 (Pin_4), J3.1 (Pin_1)
- new net GND: C2.1, C3.1, C4.1, C5.1, J1.14 (Pin_14), J1.20 (Pin_20), J1.25 (Pin_25), J1.30 (Pin_30), J1.34 (Pin_34), J1.39 (Pin_39), J1.6 (Pin_6), J1.9 (Pin_9), J2.2 (Pin_2), J3.3 (Pin_3), R1.2
- new net PIR_GPIO: J1.18 (Pin_18), R1.1, R6.1
- new net SCL: J1.5 (Pin_5), R2.1
- new net SDA: J1.3 (Pin_3), R3.1
- no-connect marks 0 -> 26
