File: Dakboard-HDMI-dimmer-KiCAD/Dakboard-HDMI-dimmer-v1/Dakboard-HDMI-dimmer-v1.kicad_pcb (KiCad board)
At the start: 2 copper layers, 30 x 65 mm, 17 parts, among them J1 Conn_02x20_Odd_Even, J2 Conn_01x05, J3 Conn_01x03

Commit message: rename
Other:
- board text added: "Dakboard-HDMI-dimmer-v1 Rev. 1 DotaPie @ May 2026"
- board text removed: "Dakboard HDMI dimmer v1 Rev. 1 DotaPie @ May 2026"
Changed lines of the file:
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@@
 		(property ki_fp_filters "MountingHole*Pad*")
 		(sheetname "/")
-		(sheetfile "Dakboard HDMI dimmer v1.kicad_sch")
+		(sheetfile "Dakboard-HDMI-dimmer-v1.kicad_sch")
 		(units
 			(unit
@@
 		(property ki_fp_filters "MountingHole*Pad*")
 		(sheetname "/")
-		(sheetfile "Dakboard HDMI dimmer v1.kicad_sch")
+		(sheetfile "Dakboard-HDMI-dimmer-v1.kicad_sch")
 		(units
 			(unit
@@
 		(property ki_fp_filters "MountingHole*Pad*")
 		(sheetname "/")
-		(sheetfile "Dakboard HDMI dimmer v1.kicad_sch")
+		(sheetfile "Dakboard-HDMI-dimmer-v1.kicad_sch")
 		(units
 			(unit
@@
 		(property ki_fp_filters "MountingHole*Pad*")
 		(sheetname "/")
-		(sheetfile "Dakboard HDMI dimmer v1.kicad_sch")
+		(sheetfile "Dakboard-HDMI-dimmer-v1.kicad_sch")
 		(units
 			(unit
@@
 		(property ki_fp_filters "C_*")
 		(sheetname "/")
-		(sheetfile "Dakboard HDMI dimmer v1.kicad_sch")
+		(sheetfile "Dakboard-HDMI-dimmer-v1.kicad_sch")
 		(units
 			(unit
@@
 		(property ki_fp_filters "Connector*:*_1x??_*")
 		(sheetname "/")
-		(sheetfile "Dakboard HDMI dimmer v1.kicad_sch")
+		(sheetfile "Dakboard-HDMI-dimmer-v1.kicad_sch")
 		(units
 			(unit
@@
 		(property ki_fp_filters "R_*")
 		(sheetname "/")
-		(sheetfile "Dakboard HDMI dimmer v1.kicad_sch")
+		(sheetfile "Dakboard-HDMI-dimmer-v1.kicad_sch")
 		(units
 			(unit
@@
 		(property ki_fp_filters "C_*")
 		(sheetname "/")
-		(sheetfile "Dakboard HDMI dimmer v1.kicad_sch")
+		(sheetfile "Dakboard-HDMI-dimmer-v1.kicad_sch")
 		(units
 			(unit
@@
 		(property ki_fp_filters "R_*")
 		(sheetname "/")
-		(sheetfile "Dakboard HDMI dimmer v1.kicad_sch")
+		(sheetfile "Dakboard-HDMI-dimmer-v1.kicad_sch")
 		(units
 			(unit
@@
 		(property ki_fp_filters "C_*")
 		(sheetname "/")
-		(sheetfile "Dakboard HDMI dimmer v1.kicad_sch")
+		(sheetfile "Dakboard-HDMI-dimmer-v1.kicad_sch")
 		(units
 			(unit
@@
 		(property ki_fp_filters "R_*")
 		(sheetname "/")
-		(sheetfile "Dakboard HDMI dimmer v1.kicad_sch")
+		(sheetfile "Dakboard-HDMI-dimmer-v1.kicad_sch")
 		(units
 			(unit
@@
 		(property ki_fp_filters "Connector*:*_2x??_*")
 		(sheetname "/")
-		(sheetfile "Dakboard HDMI dimmer v1.kicad_sch")
+		(sheetfile "Dakboard-HDMI-dimmer-v1.kicad_sch")
 		(units
 			(unit
@@
 		(property ki_fp_filters "R_*")
 		(sheetname "/")
-		(sheetfile "Dakboard HDMI dimmer v1.kicad_sch")
+		(sheetfile "Dakboard-HDMI-dimmer-v1.kicad_sch")
 		(units
 			(unit
@@
 		(property ki_fp_filters "Connector*:*_1x??_*")
 		(sheetname "/")
-		(sheetfile "Dakboard HDMI dimmer v1.kicad_sch")
+		(sheetfile "Dakboard-HDMI-dimmer-v1.kicad_sch")
 		(units
 			(unit
@@
 		(property ki_fp_filters "R_*")
 		(sheetname "/")
-		(sheetfile "Dakboard HDMI dimmer v1.kicad_sch")
+		(sheetfile "Dakboard-HDMI-dimmer-v1.kicad_sch")
 		(units
 			(unit
@@
 		(property ki_fp_filters "R_*")
 		(sheetname "/")
-		(sheetfile "Dakboard HDMI dimmer v1.kicad_sch")
+		(sheetfile "Dakboard-HDMI-dimmer-v1.kicad_sch")
 		(units
 			(unit
@@
 		(property ki_fp_filters "C_*")
 		(sheetname "/")
-		(sheetfile "Dakboard HDMI dimmer v1.kicad_sch")
+		(sheetfile "Dakboard-HDMI-dimmer-v1.kicad_sch")
 		(units
 			(unit
@@
 		(layer "Edge.Cuts")
 	)
-	(gr_text "Dakboard HDMI dimmer v1\nRev. 1\nDotaPie @ May 2026"
+	(gr_text "Dakboard-HDMI-dimmer-v1\nRev. 1\nDotaPie @ May 2026"
 		(at 126 92.25 90)
 		(layer "F.SilkS")
